Commit message: Changed default IK and added new EE to chain

File: ur_e_description/urdf/ur10e_robotiq_2f_85_robot.urdf.xacro (robot description, xacro)
@@ -28,5 +28,5 @@
     <parent link="tool0" />
     <child link = "virtual_ee_link" />
-    <origin xyz="0.0 0.0 0.1654" rpy="0.0 0.0 0.0" />
+    <origin xyz="0.0 0.0 0.1445" rpy="0.0 0.0 0.0" />
   </joint>
 </robot>
